Commit message: add real experiment and fix sim feedback parameters

File: franka_exo/robot.urdf (robot description, URDF)
Before this commit: robot franka_exo, 14 links, 13 joints
Links:
- link flange: mass 0.00663715 -> 0.0195
- link link_0: mass 0.05936 -> 0.07936
- link link_1: mass 0.0618805 -> 0.0775
- link link_2: mass 0.05754 -> 0.0444
- link link_3: mass 0.092856 -> 0.0844
- link link_4: mass 0.0504525 -> 0.039
- link link_5: mass 0.0942798 -> 0.104
- link motor540_2: mass 0.165 -> 0.173
- link motor540_4: mass 0.165 -> 0.1732
